Commit message: before teleop

File: teocart_description/urdf/teocart.xacro (robot description, xacro)
@@ -3,8 +3,5 @@
 <xacro:include filename="$(find teocart_description)/urdf/materials.xacro" />
 <xacro:include filename="$(find teocart_description)/urdf/teocart.trans" />
-<!-- <xacro:include filename="$(find teocart_description)/urdf/teocart.gazebo" /> -->
-<xacro:include filename="$(find teocart_description)/gazebo/teocart_materials.gazebo" />
-<xacro:include filename="$(find teocart_description)/gazebo/teocart_plugins.gazebo" />
-<xacro:include filename="$(find teocart_description)/gazebo/teocart_physics.gazebo" />
+<xacro:include filename="$(find teocart_description)/urdf/teocart.gazebo" />
 <link name="base_link">
   <inertial>
@@ -18,4 +15,5 @@
       <mesh filename="package://teocart_description/meshes/base_link.stl" scale="0.001 0.001 0.001"/>
     </geometry>
+    <material name="silver"/>
   </visual>
   <collision>
@@ -26,20 +24,121 @@
   </collision>
 </link>
-<link name="wheel_rod_1">
-  <inertial>
-    <origin xyz="1.4393681731971475e-07 -0.2249998739100504 -5.130204605574562e-08" rpy="0 0 0"/>
-    <mass value="0.5554849067522354"/>
-    <inertia ixx="0.009503" iyy="0.000259" izz="0.009503" ixy="0.0" iyz="-0.0" ixz="0.0"/>
-  </inertial>
-  <visual>
-    <origin xyz="-2.3e-05 -0.226142 -0.098303" rpy="0 0 0"/>
-    <geometry>
-      <mesh filename="package://teocart_description/meshes/wheel_rod_1.stl" scale="0.001 0.001 0.001"/>
-    </geometry>
-  </visual>
-  <collision>
-    <origin xyz="-2.3e-05 -0.226142 -0.098303" rpy="0 0 0"/>
-    <geometry>
-      <mesh filename="package://teocart_description/meshes/wheel_rod_1.stl" scale="0.001 0.001 0.001"/>
+<link name="Lidar_1">
+  <inertial>
+    <origin xyz="1.8157966345931263e-07 1.2608995146471194e-07 0.014555382495114899" rpy="0 0 0"/>
+    <mass value="1.142168118236333"/>
+    <inertia ixx="0.000526" iyy="0.000525" izz="0.000887" ixy="0.0" iyz="-0.0" ixz="-0.0"/>
+  </inertial>
+  <visual>
+    <origin xyz="6.4e-05 -0.001142 -0.348303" rpy="0 0 0"/>
+    <geometry>
+      <mesh filename="package://teocart_description/meshes/Lidar_1.stl" scale="0.001 0.001 0.001"/>
+    </geometry>
+    <material name="silver"/>
+  </visual>
+  <collision>
+    <origin xyz="6.4e-05 -0.001142 -0.348303" rpy="0 0 0"/>
+    <geometry>
+      <mesh filename="package://teocart_description/meshes/Lidar_1.stl" scale="0.001 0.001 0.001"/>
+    </geometry>
+  </collision>
+</link>
+<link name="front_right_caster_wheel_1">
+  <inertial>
+    <origin xyz="3.740591836276508e-09 -8.323758349249033e-12 -0.11635757818376496" rpy="0 0 0"/>
+    <mass value="5.160419362694764"/>
+    <inertia ixx="0.024515" iyy="0.024515" izz="0.002282" ixy="-0.0" iyz="0.0" ixz="-0.0"/>
+  </inertial>
+  <visual>
+    <origin xyz="-0.251 0.13 -0.243303" rpy="0 0 0"/>
+    <geometry>
+      <mesh filename="package://teocart_description/meshes/front_right_caster_wheel_1.stl" scale="0.001 0.001 0.001"/>
+    </geometry>
+    <material name="silver"/>
+  </visual>
+  <collision>
+    <origin xyz="-0.251 0.13 -0.243303" rpy="0 0 0"/>
+    <geometry>
+      <mesh filename="package://teocart_description/meshes/front_right_caster_wheel_1.stl" scale="0.001 0.001 0.001"/>
+    </geometry>
+  </collision>
+</link>
+<link name="front_left_caster_wheel_1">
+  <inertial>
+    <origin xyz="3.740592613432625e-09 1.9735255651909256e-09 -0.11635757818376496" rpy="0 0 0"/>
+    <mass value="5.160419362694764"/>
+    <inertia ixx="0.024515" iyy="0.024515" izz="0.002282" ixy="0.0" iyz="0.0" ixz="-0.0"/>
+  </inertial>
+  <visual>
+    <origin xyz="-0.251 -0.133 -0.243303" rpy="0 0 0"/>
+    <geometry>
+      <mesh filename="package://teocart_description/meshes/front_left_caster_wheel_1.stl" scale="0.001 0.001 0.001"/>
+    </geometry>
+    <material name="silver"/>
+  </visual>
+  <collision>
+    <origin xyz="-0.251 -0.133 -0.243303" rpy="0 0 0"/>
+    <geometry>
+      <mesh filename="package://teocart_description/meshes/front_left_caster_wheel_1.stl" scale="0.001 0.001 0.001"/>
+    </geometry>
+  </collision>
+</link>
+<link name="right_left_caster_wheel_1">
+  <inertial>
+    <origin xyz="4.058697822273416e-13 -8.323758349249033e-12 -0.11635757818376496" rpy="0 0 0"/>
+    <mass value="5.160419362694764"/>
+    <inertia ixx="0.024515" iyy="0.024515" izz="0.002282" ixy="0.0" iyz="0.0" ixz="0.0"/>
+  </inertial>
+  <visual>
+    <origin xyz="0.25 0.13 -0.243303" rpy="0 0 0"/>
+    <geometry>
+      <mesh filename="package://teocart_description/meshes/right_left_caster_wheel_1.stl" scale="0.001 0.001 0.001"/>
+    </geometry>
+    <material name="silver"/>
+  </visual>
+  <collision>
+    <origin xyz="0.25 0.13 -0.243303" rpy="0 0 0"/>
+    <geometry>
+      <mesh filename="package://teocart_description/meshes/right_left_caster_wheel_1.stl" scale="0.001 0.001 0.001"/>
+    </geometry>
+  </collision>
+</link>
+<link name="rear_left_caster_wheel_1">
+  <inertial>
+    <origin xyz="4.066191827689636e-13 1.9735255651909256e-09 -0.11635757818376488" rpy="0 0 0"/>
+    <mass value="5.160419362694764"/>
+    <inertia ixx="0.024515" iyy="0.024515" izz="0.002282" ixy="-0.0" iyz="0.0" ixz="-0.0"/>
+  </inertial>
+  <visual>
+    <origin xyz="0.25 -0.133 -0.243303" rpy="0 0 0"/>
+    <geometry>
+      <mesh filename="package://teocart_description/meshes/rear_left_caster_wheel_1.stl" scale="0.001 0.001 0.001"/>
+    </geometry>
+    <material name="silver"/>
+  </visual>
+  <collision>
+    <origin xyz="0.25 -0.133 -0.243303" rpy="0 0 0"/>
+    <geometry>
+      <mesh filename="package://teocart_description/meshes/rear_left_caster_wheel_1.stl" scale="0.001 0.001 0.001"/>
+    </geometry>
+  </collision>
+</link>
+<link name="camera_1">
+  <inertial>
+    <origin xyz="0.005476548100343703 0.0005884720498845288 0.001825852987195009" rpy="0 0 0"/>
+    <mass value="0.4400307041952206"/>
+    <inertia ixx="0.001023" iyy="3.8e-05" izz="0.001001" ixy="-1e-06" iyz="-0.0" ixz="8e-06"/>
+  </inertial>
+  <visual>
+    <origin xyz="-0.352673 0.0025 -0.20117" rpy="0 0 0"/>
+    <geometry>
+      <mesh filename="package://teocart_description/meshes/camera_1.stl" scale="0.001 0.001 0.001"/>
+    </geometry>
+    <material name="silver"/>
+  </visual>
+  <collision>
+    <origin xyz="-0.352673 0.0025 -0.20117" rpy="0 0 0"/>
+    <geometry>
+      <mesh filename="package://teocart_description/meshes/camera_1.stl" scale="0.001 0.001 0.001"/>
     </geometry>
   </collision>
@@ -56,4 +155,5 @@
       <mesh filename="package://teocart_description/meshes/left_wheel_1.stl" scale="0.001 0.001 0.001"/>
     </geometry>
+    <material name="silver"/>
   </visual>
   <collision>
@@ -75,4 +175,5 @@
       <mesh filename="package://teocart_description/meshes/right_wheel_1.stl" scale="0.001 0.001 0.001"/>
     </geometry>
+    <material name="silver"/>
   </visual>
   <collision>
@@ -83,164 +184,45 @@
   </collision>
 </link>
-<link name="Lidar_1">
-  <inertial>
-    <origin xyz="1.8157966345931263e-07 1.2608995146471194e-07 0.014555382495114899" rpy="0 0 0"/>
-    <mass value="1.142168118236333"/>
-    <inertia ixx="0.000526" iyy="0.000525" izz="0.000887" ixy="0.0" iyz="-0.0" ixz="-0.0"/>
-  </inertial>
-  <visual>
-    <origin xyz="6.4e-05 -0.001142 -0.348303" rpy="0 0 0"/>
-    <geometry>
-      <mesh filename="package://teocart_description/meshes/Lidar_1.stl" scale="0.001 0.001 0.001"/>
-    </geometry>
-  </visual>
-  <collision>
-    <origin xyz="6.4e-05 -0.001142 -0.348303" rpy="0 0 0"/>
-    <geometry>
-      <mesh filename="package://teocart_description/meshes/Lidar_1.stl" scale="0.001 0.001 0.001"/>
-    </geometry>
-  </collision>
-</link>
-<link name="front_right_caster_wheel_1">
-  <inertial>
-    <origin xyz="3.740591725254205e-09 -8.323675082522186e-12 -0.11691406543647123" rpy="0 0 0"/>
-    <mass value="5.185144984931505"/>
-    <inertia ixx="0.024857" iyy="0.024857" izz="0.002293" ixy="0.0" iyz="-0.0" ixz="0.0"/>
-  </inertial>
-  <visual>
-    <origin xyz="-0.251 0.13 -0.243303" rpy="0 0 0"/>
-    <geometry>
-      <mesh filename="package://teocart_description/meshes/front_right_caster_wheel_1.stl" scale="0.001 0.001 0.001"/>
-    </geometry>
-  </visual>
-  <collision>
-    <origin xyz="-0.251 0.13 -0.243303" rpy="0 0 0"/>
-    <geometry>
-      <mesh filename="package://teocart_description/meshes/front_right_caster_wheel_1.stl" scale="0.001 0.001 0.001"/>
-    </geometry>
-  </collision>
-</link>
-<link name="front_left_caster_wheel_1">
-  <inertial>
-    <origin xyz="3.740592502410323e-09 1.97352553743535e-09 -0.11691406543647123" rpy="0 0 0"/>
-    <mass value="5.185144984931505"/>
-    <inertia ixx="0.024857" iyy="0.024857" izz="0.002293" ixy="-0.0" iyz="0.0" ixz="0.0"/>
-  </inertial>
-  <visual>
-    <origin xyz="-0.251 -0.133 -0.243303" rpy="0 0 0"/>
-    <geometry>
-      <mesh filename="package://teocart_description/meshes/front_left_caster_wheel_1.stl" scale="0.001 0.001 0.001"/>
-    </geometry>
-  </visual>
-  <collision>
-    <origin xyz="-0.251 -0.133 -0.243303" rpy="0 0 0"/>
-    <geometry>
-      <mesh filename="package://teocart_description/meshes/front_left_caster_wheel_1.stl" scale="0.001 0.001 0.001"/>
-    </geometry>
-  </collision>
-</link>
-<link name="right_left_caster_wheel_1">
-  <inertial>
-    <origin xyz="4.059808045298041e-13 -8.323675082522186e-12 -0.11691406543647123" rpy="0 0 0"/>
-    <mass value="5.185144984931505"/>
-    <inertia ixx="0.024857" iyy="0.024857" izz="0.002293" ixy="-0.0" iyz="-0.0" ixz="-0.0"/>
-  </inertial>
-  <visual>
-    <origin xyz="0.25 0.13 -0.243303" rpy="0 0 0"/>
-    <geometry>
-      <mesh filename="package://teocart_description/meshes/right_left_caster_wheel_1.stl" scale="0.001 0.001 0.001"/>
-    </geometry>
-  </visual>
-  <collision>
-    <origin xyz="0.25 0.13 -0.243303" rpy="0 0 0"/>
-    <geometry>
-      <mesh filename="package://teocart_description/meshes/right_left_caster_wheel_1.stl" scale="0.001 0.001 0.001"/>
-    </geometry>
-  </collision>
-</link>
-<link name="rear_left_caster_wheel_1">
-  <inertial>
-    <origin xyz="4.0670244949581047e-13 1.97352553743535e-09 -0.11691406543647118" rpy="0 0 0"/>
-    <mass value="5.185144984931505"/>
-    <inertia ixx="0.024857" iyy="0.024857" izz="0.002293" ixy="-0.0" iyz="0.0" ixz="-0.0"/>
-  </inertial>
-  <visual>
-    <origin xyz="0.25 -0.133 -0.243303" rpy="0 0 0"/>
-    <geometry>
-      <mesh filename="package://teocart_description/meshes/rear_left_caster_wheel_1.stl" scale="0.001 0.001 0.001"/>
-    </geometry>
-  </visual>
-  <collision>
-    <origin xyz="0.25 -0.133 -0.243303" rpy="0 0 0"/>
-    <geometry>
-      <mesh filename="package://teocart_description/meshes/rear_left_caster_wheel_1.stl" scale="0.001 0.001 0.001"/>
-    </geometry>
-  </collision>
-</link>
-<link name="camera_1">
-  <inertial>
-    <origin xyz="0.005476548100343703 0.0005884720498845492 0.001825852987195009" rpy="0 0 0"/>
-    <mass value="0.4400307041952206"/>
-    <inertia ixx="0.001023" iyy="3.8e-05" izz="0.001001" ixy="-1e-06" iyz="-0.0" ixz="8e-06"/>
-  </inertial>
-  <visual>
-    <origin xyz="-0.352673 0.0025 -0.20117" rpy="0 0 0"/>
-    <geometry>
-      <mesh filename="package://teocart_description/meshes/camera_1.stl" scale="0.001 0.001 0.001"/>
-    </geometry>
-  </visual>
-  <collision>
-    <origin xyz="-0.352673 0.0025 -0.20117" rpy="0 0 0"/>
-    <geometry>
-      <mesh filename="package://teocart_description/meshes/camera_1.stl" scale="0.001 0.001 0.001"/>
-    </geometry>
-  </collision>
-</link>
-<joint name="Rigid 4" type="fixed">
+<joint name="lidar_joint" type="fixed">
+  <origin xyz="-6.4e-05 0.001142 0.348303" rpy="0 0 0"/>
+  <parent link="base_link"/>
+  <child link="Lidar_1"/>
+</joint>
+<joint name="Rigid 10" type="fixed">
+  <origin xyz="0.251 -0.13 0.243303" rpy="0 0 0"/>
+  <parent link="base_link"/>
+  <child link="front_right_caster_wheel_1"/>
+</joint>
+<joint name="Rigid 11" type="fixed">
+  <origin xyz="0.251 0.133 0.243303" rpy="0 0 0"/>
+  <parent link="base_link"/>
+  <child link="front_left_caster_wheel_1"/>
+</joint>
+<joint name="Rigid 12" type="fixed">
+  <origin xyz="-0.25 -0.13 0.243303" rpy="0 0 0"/>
+  <parent link="base_link"/>
+  <child link="right_left_caster_wheel_1"/>
+</joint>
+<joint name="Rigid 13" type="fixed">
+  <origin xyz="-0.25 0.133 0.243303" rpy="0 0 0"/>
+  <parent link="base_link"/>
+  <child link="rear_left_caster_wheel_1"/>
+</joint>
+<joint name="Rigid 14" type="fixed">
+  <origin xyz="0.352673 -0.0025 0.20117" rpy="0 0 0"/>
+  <parent link="base_link"/>
+  <child link="camera_1"/>
+</joint>
+<joint name="left_motor" type="continuous">
   <origin xyz="2.3e-05 0.226142 0.098303" rpy="0 0 0"/>
   <parent link="base_link"/>
-  <child link="wheel_rod_1"/>
-</joint>
-<joint name="left_motor" type="continuous">
-  <origin xyz="0.0 0.0 0.0" rpy="0 0 0"/>
-  <parent link="wheel_rod_1"/>
   <child link="left_wheel_1"/>
   <axis xyz="0.0 1.0 -0.0"/>
 </joint>
-<joint name="Right_motor" type="continuous">
-  <origin xyz="0.0 -0.45 0.0" rpy="0 0 0"/>
-  <parent link="wheel_rod_1"/>
+<joint name="right_motor" type="continuous">
+  <origin xyz="2.3e-05 -0.223858 0.098303" rpy="0 0 0"/>
+  <parent link="base_link"/>
   <child link="right_wheel_1"/>
-  <axis xyz="0.0 1.0 -0.0"/>
-</joint>
-<joint name="Rigid 8" type="fixed">
-  <origin xyz="-6.4e-05 0.001142 0.348303" rpy="0 0 0"/>
-  <parent link="base_link"/>
-  <child link="Lidar_1"/>
-</joint>
-<joint name="Rigid 10" type="fixed">
-  <origin xyz="0.251 -0.13 0.243303" rpy="0 0 0"/>
-  <parent link="base_link"/>
-  <child link="front_right_caster_wheel_1"/>
-</joint>
-<joint name="Rigid 11" type="fixed">
-  <origin xyz="0.251 0.133 0.243303" rpy="0 0 0"/>
-  <parent link="base_link"/>
-  <child link="front_left_caster_wheel_1"/>
-</joint>
-<joint name="Rigid 12" type="fixed">
-  <origin xyz="-0.25 -0.13 0.243303" rpy="0 0 0"/>
-  <parent link="base_link"/>
-  <child link="right_left_caster_wheel_1"/>
-</joint>
-<joint name="Rigid 13" type="fixed">
-  <origin xyz="-0.25 0.133 0.243303" rpy="0 0 0"/>
-  <parent link="base_link"/>
-  <child link="rear_left_caster_wheel_1"/>
-</joint>
-<joint name="Rigid 14" type="fixed">
-  <origin xyz="0.352673 -0.0025 0.20117" rpy="0 0 0"/>
-  <parent link="base_link"/>
-  <child link="camera_1"/>
+  <axis xyz="-0.0 -1.0 0.0"/>
 </joint>
 </robot>

Commit message: modified caster

File: teocart_description/urdf/teocart.xacro (robot description, xacro)
@@ -6,6 +6,6 @@
 <link name="base_link">
   <inertial>
-    <origin xyz="0.000985373150553865 0.0011444340597344886 0.41274312860244255" rpy="0 0 0"/>
-    <mass value="57.26708608289835"/>
+    <origin xyz="0.000985373150554124 0.0011444340597345749 0.4127431286024428" rpy="0 0 0"/>
+    <mass value="57.26708608289834"/>
     <inertia ixx="4.583669" iyy="7.340401" izz="6.097273" ixy="-4.7e-05" iyz="2.9e-05" ixz="0.012483"/>
   </inertial>
@@ -46,7 +46,7 @@
 <link name="front_right_caster_wheel_1">
   <inertial>
-    <origin xyz="3.740591836276508e-09 -8.323758349249033e-12 -0.11635757818376496" rpy="0 0 0"/>
-    <mass value="5.160419362694764"/>
-    <inertia ixx="0.024515" iyy="0.024515" izz="0.002282" ixy="-0.0" iyz="0.0" ixz="-0.0"/>
+    <origin xyz="3.740591836276508e-09 -8.323675082522186e-12 -0.11619173194709467" rpy="0 0 0"/>
+    <mass value="5.153050505798358"/>
+    <inertia ixx="0.024413" iyy="0.024413" izz="0.002279" ixy="0.0" iyz="-0.0" ixz="-0.0"/>
   </inertial>
   <visual>
@@ -66,7 +66,7 @@
 <link name="front_left_caster_wheel_1">
   <inertial>
-    <origin xyz="3.740592613432625e-09 1.9735255651909256e-09 -0.11635757818376496" rpy="0 0 0"/>
-    <mass value="5.160419362694764"/>
-    <inertia ixx="0.024515" iyy="0.024515" izz="0.002282" ixy="0.0" iyz="0.0" ixz="-0.0"/>
+    <origin xyz="3.740592613432625e-09 1.9735255096797744e-09 -0.11619173194709467" rpy="0 0 0"/>
+    <mass value="5.153050505798358"/>
+    <inertia ixx="0.024413" iyy="0.024413" izz="0.002279" ixy="0.0" iyz="0.0" ixz="-0.0"/>
   </inertial>
   <visual>
@@ -86,7 +86,7 @@
 <link name="right_left_caster_wheel_1">
   <inertial>
-    <origin xyz="4.058697822273416e-13 -8.323758349249033e-12 -0.11635757818376496" rpy="0 0 0"/>
-    <mass value="5.160419362694764"/>
-    <inertia ixx="0.024515" iyy="0.024515" izz="0.002282" ixy="0.0" iyz="0.0" ixz="0.0"/>
+    <origin xyz="4.058697822273416e-13 -8.323675082522186e-12 -0.11619173194709467" rpy="0 0 0"/>
+    <mass value="5.153050505798358"/>
+    <inertia ixx="0.024413" iyy="0.024413" izz="0.002279" ixy="-0.0" iyz="-0.0" ixz="0.0"/>
   </inertial>
   <visual>
@@ -106,7 +106,7 @@
 <link name="rear_left_caster_wheel_1">
   <inertial>
-    <origin xyz="4.066191827689636e-13 1.9735255651909256e-09 -0.11635757818376488" rpy="0 0 0"/>
-    <mass value="5.160419362694764"/>
-    <inertia ixx="0.024515" iyy="0.024515" izz="0.002282" ixy="-0.0" iyz="0.0" ixz="-0.0"/>
+    <origin xyz="4.066191827689636e-13 1.9735255096797744e-09 -0.11619173194709462" rpy="0 0 0"/>
+    <mass value="5.153050505798358"/>
+    <inertia ixx="0.024413" iyy="0.024413" izz="0.002279" ixy="-0.0" iyz="0.0" ixz="0.0"/>
   </inertial>
   <visual>
@@ -126,5 +126,5 @@
 <link name="camera_1">
   <inertial>
-    <origin xyz="0.005476548100343703 0.0005884720498845288 0.001825852987195009" rpy="0 0 0"/>
+    <origin xyz="0.005476548100343703 0.0005884720498845492 0.001825852987195009" rpy="0 0 0"/>
     <mass value="0.4400307041952206"/>
     <inertia ixx="0.001023" iyy="3.8e-05" izz="0.001001" ixy="-1e-06" iyz="-0.0" ixz="8e-06"/>

Commit message: teleop working

File: teocart_description/urdf/teocart.xacro (robot description, xacro)
@@ -3,5 +3,7 @@
 <xacro:include filename="$(find teocart_description)/urdf/materials.xacro" />
 <xacro:include filename="$(find teocart_description)/urdf/teocart.trans" />
-<xacro:include filename="$(find teocart_description)/urdf/teocart.gazebo" />
+<xacro:include filename="$(find teocart_description)/gazebo/teocart_materials.gazebo" />
+<xacro:include filename="$(find teocart_description)/gazebo/teocart_physics.gazebo" />
+<xacro:include filename="$(find teocart_description)/gazebo/teocart_plugins.gazebo" />
 <link name="base_link">
   <inertial>
@@ -224,5 +226,5 @@
   <parent link="base_link"/>
   <child link="right_wheel_1"/>
-  <axis xyz="-0.0 -1.0 0.0"/>
+  <axis xyz="-0.0 1.0 0.0"/>
 </joint>
 </robot>
